Commit message: Low poly meshes

File: src/auv_descriptions/urdf/auv_actuators.xacro (robot description, xacro)
@@ -13,6 +13,6 @@
 -->
 <robot xmlns:xacro="http://www.ros.org/wiki/xacro">
-  <xacro:property name="prop_mesh_file" value="file://$(find auv_descriptions)/meshes/prop.dae"/>
-  <xacro:property name="fin_mesh_file" value="file://$(find auv_descriptions)/meshes/fin_scaled.dae"/>
+  <xacro:property name="prop_mesh_file" value="file://$(find auv_descriptions)/meshes/prop_low.dae"/>
+  <xacro:property name="fin_mesh_file" value="file://$(find auv_descriptions)/meshes/fin_scaled_low.dae"/>
   <!-- Thruster joint and link snippet -->
   <xacro:macro name="thruster_macro"

File: src/auv_descriptions/urdf/auv_base.xacro (robot description, xacro)
@@ -12,6 +12,6 @@
   <!-- Parameters -->
   <xacro:property name="namespace" value="auv"/>
-  <xacro:property name="visual_mesh_file" value="file://$(find auv_descriptions)/meshes/auv_body.dae"/>
-  <xacro:property name="prop_mesh_file" value="file://$(find auv_descriptions)/meshes/prop.dae"/>
+  <xacro:property name="visual_mesh_file" value="file://$(find auv_descriptions)/meshes/auv_body_low.dae"/>
+  <xacro:property name="prop_mesh_file" value="file://$(find auv_descriptions)/meshes/prop_low.dae"/>
   <xacro:include filename="$(find auv_descriptions)/urdf/macros.xacro" />
   <xacro:property name="PI" value="3.14159265359"/>

Commit message: Revert "Add high waves"

File: src/auv_descriptions/urdf/auv_actuators.xacro (robot description, xacro)
@@ -13,6 +13,6 @@
 -->
 <robot xmlns:xacro="http://www.ros.org/wiki/xacro">
-  <xacro:property name="prop_mesh_file" value="file://$(find auv_descriptions)/meshes/prop_low.dae"/>
-  <xacro:property name="fin_mesh_file" value="file://$(find auv_descriptions)/meshes/fin_scaled_low.dae"/>
+  <xacro:property name="prop_mesh_file" value="file://$(find auv_descriptions)/meshes/prop.dae"/>
+  <xacro:property name="fin_mesh_file" value="file://$(find auv_descriptions)/meshes/fin_scaled.dae"/>
   <!-- Thruster joint and link snippet -->
   <xacro:macro name="thruster_macro"

File: src/auv_descriptions/urdf/auv_base.xacro (robot description, xacro)
@@ -12,6 +12,6 @@
   <!-- Parameters -->
   <xacro:property name="namespace" value="auv"/>
-  <xacro:property name="visual_mesh_file" value="file://$(find auv_descriptions)/meshes/auv_body_low.dae"/>
-  <xacro:property name="prop_mesh_file" value="file://$(find auv_descriptions)/meshes/prop_low.dae"/>
+  <xacro:property name="visual_mesh_file" value="file://$(find auv_descriptions)/meshes/auv_body.dae"/>
+  <xacro:property name="prop_mesh_file" value="file://$(find auv_descriptions)/meshes/prop.dae"/>
   <xacro:include filename="$(find auv_descriptions)/urdf/macros.xacro" />
   <xacro:property name="PI" value="3.14159265359"/>
